Commit message: Updating the meshes to split the bumper in half so we can have left and right separate detections.

File: urdf/bumper.xacro (robot description, xacro)
@@ -1,5 +1,5 @@
 <?xml version="1.0" ?>
-    <robot name="scuttle" xmlns:xacro="http://www.ros.org/wiki/xacro">
-    <link name="front_bumper_link">
+<robot name="scuttle" xmlns:xacro="http://www.ros.org/wiki/xacro">
+    <link name="front_bumper_plate_left_link">
         <inertial>
             <origin rpy="0 0 0" xyz="0 0 0"/>
@@ -10,5 +10,45 @@
             <origin rpy="0 0 0" xyz="0.10539999389648432 0 0.084749938964843793"/>
             <geometry>
-            <mesh filename="package://scuttle_model/meshes/scuttle_bumper.stl" scale="0.001 0.001 0.001"/>
+            <mesh filename="package://scuttle_bumper/meshes/scuttle_bumper_plate_left.stl" scale="0.001 0.001 0.001"/>
+            </geometry>
+            <material name="silver"/>
+        </visual>
+        <collision name="front_bumper_plate_left_link">
+            <origin rpy="0 0 0" xyz="0.10539999389648432 0 0.084749938964843793"/>
+            <geometry>
+            <mesh filename="package://scuttle_bumper/meshes/scuttle_bumper_plate_left.stl" scale="0.001 0.001 0.001"/>
+            </geometry>
+        </collision>
+    </link>
+    <link name="front_bumper_plate_right_link">
+        <inertial>
+            <origin rpy="0 0 0" xyz="0 0 0"/>
+            <mass value="0.1"/>
+            <inertia ixx="0.038876" ixy="1.3e-05" ixz="1e-06" iyy="0.047513" iyz="0.000486" izz="0.084083"/>
+        </inertial>
+        <visual>
+            <origin rpy="0 0 0" xyz="0.10539999389648432 0 0.084749938964843793"/>
+            <geometry>
+            <mesh filename="package://scuttle_bumper/meshes/scuttle_bumper_plate_right.stl" scale="0.001 0.001 0.001"/>
+            </geometry>
+            <material name="silver"/>
+        </visual>
+        <collision name="front_bumper_plate_right_link">
+            <origin rpy="0 0 0" xyz="0.10539999389648432 0 0.084749938964843793"/>
+            <geometry>
+            <mesh filename="package://scuttle_bumper/meshes/scuttle_bumper_plate_right.stl" scale="0.001 0.001 0.001"/>
+            </geometry>
+        </collision>
+    </link>
+    <link name="front_bumper_bracket_left_link">
+        <inertial>
+            <origin rpy="0 0 0" xyz="0 0 0"/>
+            <mass value="0.1"/>
+            <inertia ixx="0.038876" ixy="1.3e-05" ixz="1e-06" iyy="0.047513" iyz="0.000486" izz="0.084083"/>
+        </inertial>
+        <visual>
+            <origin rpy="0 0 0" xyz="0.10539999389648432 0 0.084749938964843793"/>
+            <geometry>
+            <mesh filename="package://scuttle_bumper/meshes/scuttle_bumper_bracket_left.stl" scale="0.001 0.001 0.001"/>
             </geometry>
             <material name="silver"/>
@@ -17,12 +57,47 @@
             <origin rpy="0 0 0" xyz="0.10539999389648432 0 0.084749938964843793"/>
             <geometry>
-            <mesh filename="package://scuttle_model/meshes/scuttle_bumper_collision_1.stl" scale="0.001 0.001 0.001"/>
+            <mesh filename="package://scuttle_bumper/meshes/scuttle_bumper_bracket_left_collision.stl" scale="0.001 0.001 0.001"/>
             </geometry>
         </collision>
     </link>
-    <joint name="front_bumper_joint" type="fixed">
+    <link name="front_bumper_bracket_right_link">
+        <inertial>
+            <origin rpy="0 0 0" xyz="0 0 0"/>
+            <mass value="0.1"/>
+            <inertia ixx="0.038876" ixy="1.3e-05" ixz="1e-06" iyy="0.047513" iyz="0.000486" izz="0.084083"/>
+        </inertial>
+        <visual>
+            <origin rpy="0 0 0" xyz="0.10539999389648432 0 0.084749938964843793"/>
+            <geometry>
+            <mesh filename="package://scuttle_bumper/meshes/scuttle_bumper_bracket_right.stl" scale="0.001 0.001 0.001"/>
+            </geometry>
+            <material name="silver"/>
+        </visual>
+        <collision>
+            <origin rpy="0 0 0" xyz="0.10539999389648432 0 0.084749938964843793"/>
+            <geometry>
+            <mesh filename="package://scuttle_bumper/meshes/scuttle_bumper_bracket_right_collision.stl" scale="0.001 0.001 0.001"/>
+            </geometry>
+        </collision>
+    </link>
+    <joint name="front_bumper_bracket_left_joint" type="fixed">
         <origin rpy="0 0 0" xyz="0.0 0.0 0.0"/>
         <parent link="base_link"/>
-        <child link="front_bumper_link"/>
+        <child link="front_bumper_bracket_left_link"/>
+    </joint>
+    <joint name="front_bumper_bracket_right_joint" type="fixed">
+        <origin rpy="0 0 0" xyz="0.0 0.0 0.0"/>
+        <parent link="base_link"/>
+        <child link="front_bumper_bracket_right_link"/>
+    </joint>
+    <joint name="front_bumper_plate_left_joint" type="fixed">
+        <origin rpy="0 0 0" xyz="0.0 0.0 0.0"/>
+        <parent link="front_bumper_bracket_left_link"/>
+        <child link="front_bumper_plate_left_link"/>
+    </joint>
+    <joint name="front_bumper_plate_right_joint" type="fixed">
+        <origin rpy="0 0 0" xyz="0.0 0.0 0.0"/>
+        <parent link="front_bumper_bracket_right_link"/>
+        <child link="front_bumper_plate_right_link"/>
     </joint>
 </robot>

Commit message: Updating the bumper sensor references

File: urdf/bumper.xacro (robot description, xacro)
@@ -15,5 +15,5 @@
             <material name="silver"/>
         </visual>
-        <collision name="front_bumper_plate_left_link">
+        <collision name="front_bumper_plate_left_cl">
             <origin rpy="0 0 0" xyz="0.10539999389648432 0 0.084749938964843793"/>
             <geometry>
@@ -35,5 +35,5 @@
             <material name="silver"/>
         </visual>
-        <collision name="front_bumper_plate_right_link">
+        <collision name="front_bumper_plate_right_cl">
             <origin rpy="0 0 0" xyz="0.10539999389648432 0 0.084749938964843793"/>
             <geometry>

Commit message: Updating the way the xacro is layed out
Unifying the meshes for the bracket and setting all frames relative to the parent frame.

File: urdf/bumper.xacro (robot description, xacro)
@@ -2,103 +2,119 @@
 <robot name="scuttle" xmlns:xacro="http://www.ros.org/wiki/xacro">
     <xacro:include filename="$(find scuttle_bumper)/urdf/bumper.gazebo" />
-    <link name="front_bumper_plate_left_link">
-        <inertial>
-            <origin rpy="0 0 0" xyz="0 0 0"/>
-            <mass value="0.1"/>
-            <inertia ixx="0.038876" ixy="1.3e-05" ixz="1e-06" iyy="0.047513" iyz="0.000486" izz="0.084083"/>
-        </inertial>
+    <!--
+        Left hand bumper elements
+    -->
+    <joint name="front_bumper_bracket_left_joint" type="fixed">
+        <origin rpy="0 0 0" xyz="0.2005 0.1375 0.015"/>
+        <parent link="chassis_link"/>
+        <child link="front_bumper_bracket_left_link"/>
+    </joint>
+    <!--
+        Define the left hand-side bumper bracket.
+    -->
+    <link name="front_bumper_bracket_left_link">
         <visual>
-            <origin rpy="0 0 0" xyz="0.10539999389648432 0 0.084749938964843793"/>
+            <origin rpy="0 0 0" xyz="0.0 0.0 0.0"/>
             <geometry>
-            <mesh filename="package://scuttle_bumper/meshes/scuttle_bumper_plate_left.stl" scale="0.001 0.001 0.001"/>
+                <mesh filename="package://scuttle_bumper/meshes/scuttle_bumper_bracket.stl" scale="0.001 0.001 0.001"/>
             </geometry>
             <material name="silver"/>
         </visual>
-        <collision name="front_bumper_plate_left_cl">
-            <origin rpy="0 0 0" xyz="0.10539999389648432 0 0.084749938964843793"/>
+        <collision>
+            <origin rpy="0 0 0" xyz="0 0 0 "/>
             <geometry>
-            <mesh filename="package://scuttle_bumper/meshes/scuttle_bumper_plate_left.stl" scale="0.001 0.001 0.001"/>
+            <mesh filename="package://scuttle_bumper/meshes/scuttle_bumper_bracket_collision.stl" scale="0.001 0.001 0.001"/>
             </geometry>
         </collision>
     </link>
+     <joint name="front_bumper_plate_left_joint" type="fixed">
+        <origin rpy="0 0 0" xyz="0.0135 -0.0225 -0.038"/>
+        <parent link="front_bumper_bracket_left_link"/>
+        <child link="front_bumper_plate_left_link"/>
+    </joint>
+    <!--
+        Define the left hand-side of the bumper plate, i.e. the part that is hit when scuttle bumps into an obstacle.
+        For URDF purposes we assume the bumper plate is split into a left-hand side and a right-hand side. In reality
+        there is only one plate but it is able to move relatively independent between the left and right hand sides.
+    -->
+    <link
+        name="front_bumper_plate_left_link">
+        <visual>
+            <origin rpy="0 0 0" xyz="0 0 0"/>
+            <geometry>
+            <!-- Link to the visual mesh and indicate that the unit of length for the mesh is millimeters. -->
+            <mesh
+                filename="package://scuttle_bumper/meshes/scuttle_bumper_plate_left.stl"
+                scale="0.001 0.001 0.001"/>
+            </geometry>
+            <material
+                name="silver"/>
+        </visual>
+        <collision
+            name="front_bumper_plate_left_cl">
+            <origin
+                rpy="0 0 0"
+                xyz="0 0 0"/>
+            <geometry>
+            <!-- Link to the collision mesh and indicate that the unit of length for the mesh is millimeters. -->
+            <mesh
+                filename="package://scuttle_bumper/meshes/scuttle_bumper_plate_left.stl"
+                scale="0.001 0.001 0.001"/>
+            </geometry>
+        </collision>
+    </link>
+    <!--
+        Right hand bumper elements
+    -->
+    <joint name="front_bumper_bracket_right_joint" type="fixed">
+        <origin rpy="0 0 0" xyz="0.2005 -0.1375 0.015"/>
+        <parent link="chassis_link"/>
+        <child link="front_bumper_bracket_right_link"/>
+    </joint>
+    <link name="front_bumper_bracket_right_link">
+       <visual>
+            <origin rpy="0 0 0" xyz="0.0 0.0 0.0"/>
+            <geometry>
+            <mesh filename="package://scuttle_bumper/meshes/scuttle_bumper_bracket.stl" scale="0.001 0.001 0.001"/>
+            </geometry>
+            <material name="silver"/>
+        </visual>
+        <collision>
+            <origin rpy="0 0 0" xyz="0 0 0"/>
+            <geometry>
+            <mesh filename="package://scuttle_bumper/meshes/scuttle_bumper_bracket_collision.stl" scale="0.001 0.001 0.001"/>
+            </geometry>
+        </collision>
+    </link>
+    <joint name="front_bumper_plate_right_joint" type="fixed">
+        <origin rpy="0 0 0" xyz="0.0135 0.0225 -0.038"/>
+        <parent link="front_bumper_bracket_right_link"/>
+        <child link="front_bumper_plate_right_link"/>
+    </joint>
+    <!--
+        Define the right hand-side of the bumper plate, i.e. the part that is hit when scuttle bumps into an obstacle.
+        For URDF purposes we assume the bumper plate is split into a left-hand side and a right-hand side. In reality
+        there is only one plate but it is able to move relatively independent between the left and right hand sides.
+    -->
     <link name="front_bumper_plate_right_link">
-        <inertial>
+        <visual>
             <origin rpy="0 0 0" xyz="0 0 0"/>
-            <mass value="0.1"/>
-            <inertia ixx="0.038876" ixy="1.3e-05" ixz="1e-06" iyy="0.047513" iyz="0.000486" izz="0.084083"/>
-        </inertial>
-        <visual>
-            <origin rpy="0 0 0" xyz="0.10539999389648432 0 0.084749938964843793"/>
             <geometry>
-            <mesh filename="package://scuttle_bumper/meshes/scuttle_bumper_plate_right.stl" scale="0.001 0.001 0.001"/>
+            <!-- Link to the visual mesh and indicate that the unit of length for the mesh is millimeters. -->
+            <mesh
+                filename="package://scuttle_bumper/meshes/scuttle_bumper_plate_right.stl"
+                scale="0.001 0.001 0.001"/>
             </geometry>
             <material name="silver"/>
         </visual>
         <collision name="front_bumper_plate_right_cl">
-            <origin rpy="0 0 0" xyz="0.10539999389648432 0 0.084749938964843793"/>
+            <origin rpy="0 0 0" xyz="0 0 0"/>
             <geometry>
-            <mesh filename="package://scuttle_bumper/meshes/scuttle_bumper_plate_right.stl" scale="0.001 0.001 0.001"/>
+            <!-- Link to the collision mesh and indicate that the unit of length for the mesh is millimeters. -->
+            <mesh
+                filename="package://scuttle_bumper/meshes/scuttle_bumper_plate_right.stl"
+                scale="0.001 0.001 0.001"/>
             </geometry>
         </collision>
     </link>
-    <link name="front_bumper_bracket_left_link">
-        <inertial>
-            <origin rpy="0 0 0" xyz="0 0 0"/>
-            <mass value="0.1"/>
-            <inertia ixx="0.038876" ixy="1.3e-05" ixz="1e-06" iyy="0.047513" iyz="0.000486" izz="0.084083"/>
-        </inertial>
-        <visual>
-            <origin rpy="0 0 0" xyz="0.10539999389648432 0 0.084749938964843793"/>
-            <geometry>
-            <mesh filename="package://scuttle_bumper/meshes/scuttle_bumper_bracket_left.stl" scale="0.001 0.001 0.001"/>
-            </geometry>
-            <material name="silver"/>
-        </visual>
-        <collision>
-            <origin rpy="0 0 0" xyz="0.10539999389648432 0 0.084749938964843793"/>
-            <geometry>
-            <mesh filename="package://scuttle_bumper/meshes/scuttle_bumper_bracket_left_collision.stl" scale="0.001 0.001 0.001"/>
-            </geometry>
-        </collision>
-    </link>
-    <link name="front_bumper_bracket_right_link">
-        <inertial>
-            <origin rpy="0 0 0" xyz="0 0 0"/>
-            <mass value="0.1"/>
-            <inertia ixx="0.038876" ixy="1.3e-05" ixz="1e-06" iyy="0.047513" iyz="0.000486" izz="0.084083"/>
-        </inertial>
-        <visual>
-            <origin rpy="0 0 0" xyz="0.10539999389648432 0 0.084749938964843793"/>
-            <geometry>
-            <mesh filename="package://scuttle_bumper/meshes/scuttle_bumper_bracket_right.stl" scale="0.001 0.001 0.001"/>
-            </geometry>
-            <material name="silver"/>
-        </visual>
-        <collision>
-            <origin rpy="0 0 0" xyz="0.10539999389648432 0 0.084749938964843793"/>
-            <geometry>
-            <mesh filename="package://scuttle_bumper/meshes/scuttle_bumper_bracket_right_collision.stl" scale="0.001 0.001 0.001"/>
-            </geometry>
-        </collision>
-    </link>
-    <joint name="front_bumper_bracket_left_joint" type="fixed">
-        <origin rpy="0 0 0" xyz="0.0 0.0 0.0"/>
-        <parent link="base_link"/>
-        <child link="front_bumper_bracket_left_link"/>
-    </joint>
-    <joint name="front_bumper_bracket_right_joint" type="fixed">
-        <origin rpy="0 0 0" xyz="0.0 0.0 0.0"/>
-        <parent link="base_link"/>
-        <child link="front_bumper_bracket_right_link"/>
-    </joint>
-    <joint name="front_bumper_plate_left_joint" type="fixed">
-        <origin rpy="0 0 0" xyz="0.0 0.0 0.0"/>
-        <parent link="front_bumper_bracket_left_link"/>
-        <child link="front_bumper_plate_left_link"/>
-    </joint>
-    <joint name="front_bumper_plate_right_joint" type="fixed">
-        <origin rpy="0 0 0" xyz="0.0 0.0 0.0"/>
-        <parent link="front_bumper_bracket_right_link"/>
-        <child link="front_bumper_plate_right_link"/>
-    </joint>
 </robot>
